Commit message: meshes

File: aiot_ws/src/move_turtle/urdf/visual.urdf (robot description, URDF)
Before this commit: robot myfirst, 9 links, 8 joints
Links:
- added link box; visual box size=0.08 0.08 0.08
- added link gipper_pole; visual cylinder length=0.2 radius=0.01
- added link head; visual sphere radius=0.2
- added link left_gipper; visual mesh filename=package://move_turtle/meshes/l_finger.dae
- added link left_tip; visual mesh filename=package://move_turtle/meshes/l_finger_tip.dae
- added link right_gipper; visual mesh filename=package://move_turtle/meshes/l_finger.dae
- added link right_tip; visual mesh filename=package://move_turtle/meshes/l_finger_tip.dae
Joints:
- added joint gripper_extension: type fixed, parent base_link, child gripper_pole, origin xyz=0.19 0 0.2 rpy=0 0 0
- added joint head_swivel: type fixed, parent base_link, child head, origin xyz=0 0 0.3
- added joint left_gripper_joint: type fixed, parent gripper_pole, child left_gripper, origin xyz=0.2 0.01 0 rpy=0 0 0
- added joint left_tip_joint: type fixed, parent left_gripper, child left_tip
- added joint right_gripper_joint: type fixed, parent gripper_pole, child right_gripper, origin xyz=0.2 -0.01 0 rpy=0 0 0
- added joint right_tip_joint: type fixed, parent right_gripper, child right_tip
- added joint tobox: type fixed, parent head, child box, origin xyz=0.1814 0 0.1414

Commit message: visual

File: aiot_ws/src/move_turtle/urdf/visual.urdf (robot description, URDF)
Before this commit: robot myfirst, 16 links, 15 joints
Links:
- removed link gipper_pole
- removed link left_gipper
- removed link right_gipper
- added link gripper_pole; visual cylinder length=0.2 radius=0.01
- added link left_gripper; visual mesh filename=package://urdf_tutorial/meshes/l_finger.dae
- added link right_gripper; visual mesh filename=package://urdf_tutorial/meshes/l_finger.dae
- link left_tip: geometry visual mesh filename=package://urdf_tutorial/meshes/l_finger_tip.dae
- link right_tip: geometry visual mesh filename=package://urdf_tutorial/meshes/l_finger_tip.dae
Joints:
- joint left_back_wheel_joint: origin xyz=-0.133 0 -0.085 -> xyz=-0.133333333333 0 -0.085 rpy=0 0 0
- joint left_base_joint: origin xyz=0.0 0 -0.6 -> xyz=0 0 -0.6
- joint left_front_wheel_joint: origin xyz=0.133 0 -0.085 -> xyz=0.133333333333 0 -0.085 rpy=0 0 0
- joint right_back_wheel_joint: origin xyz=-0.133 0 -0.085 -> xyz=-0.133333333333 0 -0.085 rpy=0 0 0
- joint right_base_joint: origin xyz=0.0 0 -0.6 -> xyz=0 0 -0.6
- joint right_front_wheel_joint: origin xyz=0.133 0 -0.085 -> xyz=0.133333333333 0 -0.085 rpy=0 0 0

Commit message: aa

File: aiot_ws/src/move_turtle/urdf/visual.urdf (robot description, URDF)
Before this commit: robot visual, 16 links, 15 joints
Links:
- link left_gripper: geometry visual mesh filename=package://move_turtle/meshes/l_finger.dae
- link left_tip: geometry visual mesh filename=package://move_turtle/meshes/l_finger_tip.dae
- link right_gripper: geometry visual mesh filename=package://move_turtle/meshes/l_finger.dae
- link right_tip: geometry visual mesh filename=package://move_turtle/meshes/l_finger_tip.dae
