Commit message: camera macroed.urdf.xacro

File: aiot_ws/src/move_turtle/urdf/macroed.urdf.xacro (robot description, xacro)
@@ -212,3 +212,25 @@
     <origin xyz="${.707*width+0.04} 0 ${.707*width}"/>
   </joint>
+  <link name="camera_link">
+    <visual>
+      <geometry>
+        <box size="0.01 0.03 0.03"/>
+      </geometry>
+      <material name="black"/>
+    </visual>
+  </link>
+  <joint name="camera_joint" type="fixed">
+    <parent link="box"/>
+    <child link="camera_link"/>
+    <origin xyz="0 0 0.04" rpy="0 0 0"/>
+  </joint>
+  <gazebo reference="camera_link">
+    <material>Gazebo/Red</material>
+  </gazebo>
+  <joint name="camera_optical_joint" type="fixed">
+    <origin xyz="0 0 0" rpy="${-pi/2} 0 ${-pi/2}"/>
+    <parent link="camera_link"/>
+    <child link= "camera_link_optical"/>
+  </joint>
+  <link name="camera_link-optical"/>
 </robot>

Commit message: aa

File: aiot_ws/src/move_turtle/urdf/macroed.urdf.xacro (robot description, xacro)
@@ -139,10 +139,10 @@
         <origin rpy="${(reflect-1)/2*pi} 0 0" xyz="0 0 0"/>
         <geometry>
-          <mesh filename="package://urdf_tutorial/meshes/l_finger.dae"/>
-        </geometry>
-      </visual>
-      <collision>
-        <geometry>
-          <mesh filename="package://urdf_tutorial/meshes/l_finger.dae"/>
+          <mesh filename="package://move_turtle/meshes/l_finger.dae"/>
+        </geometry>
+      </visual>
+      <collision>
+        <geometry>
+          <mesh filename="package://move_turtle/meshes/l_finger.dae"/>
         </geometry>
         <origin rpy="${(reflect-1)/2*pi} 0 0" xyz="0 0 0"/>
@@ -158,10 +158,10 @@
         <origin rpy="${(reflect-1)/2*pi} 0 0" xyz="0.09137 0.00495 0"/>
         <geometry>
-          <mesh filename="package://urdf_tutorial/meshes/l_finger_tip.dae"/>
-        </geometry>
-      </visual>
-      <collision>
-        <geometry>
-          <mesh filename="package://urdf_tutorial/meshes/l_finger_tip.dae"/>
+          <mesh filename="package://move_turtle/meshes/l_finger_tip.dae"/>
+        </geometry>
+      </visual>
+      <collision>
+        <geometry>
+          <mesh filename="package://move_turtle/meshes/l_finger_tip.dae"/>
         </geometry>
         <origin rpy="${(reflect-1)/2*pi} 0 0" xyz="0.09137 0.00495 0"/>
@@ -233,4 +233,4 @@
     <child link= "camera_link_optical"/>
   </joint>
-  <link name="camera_link-optical"/>
+  <link name="camera_link_optical"/>
 </robot>
